Commit message: Publish standard ROS pose and twist messages; separate button events.
* Use standard ROS messages for publishing pose and twist. This makes
  visualization easier, and gives greater compatibility.
* To improve performance with fast loop rates, use wait-free ringbuffer
  instead of blocking on mutexes.
* Prefix transform names with "geotouch" to avoid name clashes.

File: geomagic_description/urdf/omni.urdf (robot description, URDF)
Before this commit: robot geomagic_touch, 7 links, 6 joints
Joints:
- removed joint elbow
- removed joint pitch
- removed joint roll
- removed joint shoulder
- removed joint waist
- removed joint yaw
- added joint geotouch_elbow: type revolute, parent upper_arm, child lower_arm, origin xyz=0.0075 .134 0 rpy=-1.5 0 0, axis 1 0 0, limit lower=-0.81 upper=1.25 effort=5 velocity=100
- added joint geotouch_pitch: type revolute, parent wrist, child tip, origin xyz=0 0.0525 0 rpy=0.5 0 0, axis 1 0 0, limit lower=-0.5 upper=1.75 effort=5 velocity=100
- added joint geotouch_roll: type revolute, parent tip, child stylus, origin xyz=0 -0.023 0 rpy=3.14159 3.14159 0, axis 0 1 0, limit lower=-2.58 upper=2.58 effort=5 velocity=100
- added joint geotouch_shoulder: type revolute, parent torso, child upper_arm, origin xyz=-0.0075 0 0.035 rpy=0 0 0, axis 1 0 0, limit lower=0 upper=1.75 effort=5 velocity=100
- added joint geotouch_waist: type revolute, parent base, child torso, origin xyz=0 0 0.09 rpy=0 0 0, axis 0 0 1, limit lower=-0.98 upper=0.98 effort=5 velocity=100
- added joint geotouch_yaw: type revolute, parent lower_arm, child wrist, origin xyz=0 0.08 0, axis 0 1 0, limit lower=3.92 upper=8.83 effort=5 velocity=100
